Commit message: fix: added imu lidar diff-driveplugin and updated to skid steer drive

File: amr_description/models/amr/amr.xacro (robot description, xacro)
@@ -1,65 +1,49 @@
-<?xml version="1.0"?>
+<?xml version="1.0" ?>
 <!--
 *****************************************************************************************
 *
 *  Filename:			  amr.xacro
-*  Created:				  08/01/202$
-*  Last Modified:	  08/01/2024
+*  Created:				  08/01/2024
+*  Last Modified:	  15/03/2024
 *  Author:				  Archit Jain
 *
 *****************************************************************************************
 -->
-<robot name="amr" xmlns:xacro="http://www.ros.org/wiki/xacro">
+<robot name="amr" xmlns:xacro="http://ros.org/wiki/xacro">
+  <!-- ****************** INCLUDE EXTERNAL FILES *******************************  -->
   <xacro:include filename="$(find amr_description)/models/amr/amr.gazebo" />
   <xacro:include filename="$(find amr_description)/models/amr/materials.xacro" />
-  <!-- ****************** BASIC INERTIAL MACROS ***************************  -->
-  <!-- Define intertial property macros  -->
-  <xacro:macro name="box_inertia" params="m w h d *origin">
+  <!-- ****************** ROBOT CONSTANTS *******************************  -->
+  <xacro:property name="base_width" value="0.39"/>
+  <xacro:property name="base_length" value="0.70"/>
+  <xacro:property name="base_height" value="0.20"/>
+  <xacro:property name="wheel_radius" value="0.14"/>
+  <xacro:property name="wheel_width" value="0.06"/>
+  <xacro:property name="wheel_ygap" value="0.035"/>
+  <xacro:property name="wheel_zoff" value="0.05"/>
+  <xacro:property name="wheel_xoff" value="0.221"/>
+  <!-- ****************** INERTIAL PROPERTY MACROS *******************************  -->
+  <xacro:macro name="box_inertia" params="m w h d">
     <inertial>
-      <xacro:insert_block name="origin"/>
+      <origin xyz="0 0 0" rpy="${pi/2} 0 ${pi/2}"/>
       <mass value="${m}"/>
-      <inertia  ixx="${(m/12) * (h*h + d*d)}" ixy="0.0" ixz="0.0"
-                iyy="${(m/12) * (w*w + d*d)}" iyz="0.0"
-                izz="${(m/12) * (w*w + h*h)}"/>
+      <inertia ixx="${(m/12) * (h*h + d*d)}" ixy="0.0" ixz="0.0" iyy="${(m/12) * (w*w + d*d)}" iyz="0.0" izz="${(m/12) * (w*w + h*h)}"/>
     </inertial>
   </xacro:macro>
-  <xacro:macro name="cylinder_inertia" params="m r h *origin">
+  <xacro:macro name="cylinder_inertia" params="m r h">
     <inertial>
-      <xacro:insert_block name="origin"/>
+      <origin xyz="0 0 0" rpy="${pi/2} 0 0" />
       <mass value="${m}"/>
-      <inertia  ixx="${(m/12) * (3*r*r + h*h)}" ixy = "0" ixz = "0"
-                iyy="${(m/12) * (3*r*r + h*h)}" iyz = "0"
-                izz="${(m/2) * (r*r)}"/>
+      <inertia ixx="${(m/12) * (3*r*r + h*h)}" ixy = "0" ixz = "0" iyy="${(m/12) * (3*r*r + h*h)}" iyz = "0" izz="${(m/2) * (r*r)}"/>
     </inertial>
   </xacro:macro>
-  <xacro:macro name="sphere_inertia" params="m r *origin">
+  <xacro:macro name="sphere_inertia" params="m r">
     <inertial>
-      <xacro:insert_block name="origin"/>
       <mass value="${m}"/>
-      <inertia  ixx="${(2/5) * m * (r*r)}" ixy="0.0" ixz="0.0"
-                iyy="${(2/5) * m * (r*r)}" iyz="0.0"
-                izz="${(2/5) * m * (r*r)}"/>
+      <inertia ixx="${(2/5) * m * (r*r)}" ixy="0.0" ixz="0.0" iyy="${(2/5) * m * (r*r)}" iyz="0.0" izz="${(2/5) * m * (r*r)}"/>
     </inertial>
   </xacro:macro>
-  <!-- ****************** ROBOT CONSTANTS *******************************  -->
-  <!-- Define the size of the robot's main chassis in meters -->
-  <xacro:property name="amr_base_width" value="0.30"/>
-  <xacro:property name="amr_base_height" value="0.05"/>
-  <xacro:property name="amr_base_length" value="0.40"/>
-  <xacro:property name="amr_base_mass" value="1500"/>
-  <xacro:property name="wheel_radius" value="0.05" />
-  <xacro:property name="wheel_width" value="0.015" />
-  <xacro:property name="wheel_mass" value="150" />
-  <xacro:property name="wheel_zoff" value="0.025"/>    <!-- Set wheel Z offset to 0 to align wheel axis to AMR base -->
-  <xacro:property name="caster_wheel_mass" value="10" />
-  <xacro:property name="lidar_radius" value="0.05" />
-  <xacro:property name="lidar_height" value="0.04" />
-  <xacro:property name="lidar_mass" value="100" />
-  <xacro:property name="pi_2" value="1.5707963267949" />
-  <!-- <xacro:property name="pi" value="3.141592654" /> -->
   <!-- ****************** ROBOT BASE FOOTPRINT ***************************  -->
-  <!-- Define the center of the main robot chassis projected on the ground -->
   <link name="base_footprint"/>
-  <!-- The base footprint of the robot is located underneath the chassis -->
   <joint name="base_joint" type="fixed">
     <parent link="base_footprint"/>
@@ -67,155 +51,79 @@
     <origin xyz="0.0 0.0 ${(wheel_radius+wheel_zoff)}" rpy="0 0 0"/>
   </joint>
-  <!-- ****************** ROBOT BASE LINK ***************************  -->
-  <link name="base_link"/>
-  <!-- The base link of the robot is located on the chassis -->
-  <joint name="base_link_joint" type="fixed">
-    <origin xyz="0.0 0.0 0.0" rpy="0 0 0"/>
-    <parent link="base_link"/>
-    <child link="amr_base" />
-  </joint>
-  <!-- ********************** AMR BASE *********************************  -->
-  <link name="amr_base">
+  <!-- ********************** ROBOT BASE *********************************  -->
+  <link name="base_link">
     <visual>
-      <origin xyz="0 0 0" rpy="0 0 0"/>
+      <origin xyz="0 0 -0.05" rpy="1.5707963267949 0 3.141592654"/>
       <geometry>
-        <box size="${amr_base_length} ${amr_base_width} ${amr_base_height}"/>
+        <box size="${base_length} ${base_height} ${base_width}"/>
       </geometry>
-      <material name="blue" />
     </visual>
     <collision>
-      <origin xyz="0 0 0" rpy="0 0 0"/>
       <geometry>
-        <box size="${amr_base_length} ${amr_base_width} ${amr_base_height}"/>
+        <box size="${base_length} ${base_width} ${base_height}"/>
       </geometry>
     </collision>
-    <xacro:box_inertia m="${amr_base_mass}" w="${amr_base_width}" d="${amr_base_length}" h="${amr_base_height}">
-      <origin xyz="0 0 0" rpy="${pi_2} 0 ${pi_2}"/>
-    </xacro:box_inertia>
+    <xacro:box_inertia m="40.0" w="${base_width}" d="${base_length}" h="${base_height}"/>
   </link>
-  <!-- ********************** AMR LEFT WHEEL JOINT *********************************  -->
-  <joint name="amr_LW_joint" type="continuous">
-      <parent link="amr_base"/>
-      <child link="amr_LW"/>
-      <origin xyz="0.0 ${-amr_base_width/2 - wheel_width/2} ${-wheel_zoff}" rpy="0 0 0"/>
+  <!-- *********************** DRIVE WHEELS ******************************  -->
+  <xacro:macro name="wheel" params="prefix x_reflect y_reflect">
+    <link name="${prefix}_link">
+      <visual>
+        <origin xyz="0 0 0" rpy="1.5707963267949 0 0"/>
+        <geometry>
+            <cylinder radius="${wheel_radius}" length="${wheel_width}"/>
+        </geometry>
+      </visual>
+      <collision>
+        <origin xyz="0 0 0" rpy="${pi/2} 0 0"/>
+        <geometry>
+          <cylinder radius="${wheel_radius}" length="${wheel_width}"/>
+        </geometry>
+      </collision>
+      <xacro:cylinder_inertia m="110.5" r="${wheel_radius}" h="${wheel_width}"/>
+    </link>
+    <joint name="${prefix}_joint" type="revolute">
+      <parent link="base_link"/>
+      <child link="${prefix}_link"/>
+      <origin xyz="${x_reflect*wheel_xoff} ${y_reflect*(base_width/2+wheel_ygap)} ${-wheel_zoff}" rpy="0 0 0"/>
+      <limit upper="3.1415" lower="-3.1415" effort="30" velocity="5.0"/>
       <axis xyz="0 1 0"/>
+    </joint>
+  </xacro:macro>
+  <xacro:wheel prefix="drive_r_whl_l" x_reflect="-1" y_reflect="1" />
+  <xacro:wheel prefix="drive_r_whl_r" x_reflect="-1" y_reflect="-1" />
+  <xacro:wheel prefix="drive_f_whl_l" x_reflect="1" y_reflect="1" />
+  <xacro:wheel prefix="drive_f_whl_r" x_reflect="1" y_reflect="-1" />
+  <!-- *********************** IMU SETUP *********************************  -->
+  <joint name="imu_joint" type="fixed">
+    <parent link="base_link"/>
+    <child link="imu_link"/>
+    <origin xyz="-0.10 0 0.05" rpy="0 0 0"/>
   </joint>
-  <!-- ********************** AMR LEFT WHEEL *********************************  -->
-  <link name="amr_LW">
+  <link name="imu_link"/>
+  <!-- *********************** LIDAR SETUP **********************************  -->
+  <joint name="lidar_joint" type="fixed">
+    <parent link="base_link"/>
+    <child link="lidar_link"/>
+    <origin xyz="0.215 0 0.11" rpy="0 0 0"/>
+  </joint>
+  <link name="lidar_link">
+    <collision>
+     <origin xyz="0 0 0" rpy="0 0 0"/>
+     <geometry>
+      <cylinder radius="0.0508" length="0.12"/>
+     </geometry>
+    </collision>
     <visual>
-      <origin xyz="0 0 0" rpy="${pi_2} 0 0"/>
-      <geometry>
-        <cylinder radius="${wheel_radius}" length="${wheel_width}"/>
-      </geometry>
-      <material name="red" />
+     <origin xyz="0 0 0" rpy="0 0 0"/>
+     <geometry>
+      <cylinder radius="0.0508" length="0.12"/>
+     </geometry>
     </visual>
-    <collision>
-      <origin xyz="0 0 0" rpy="${pi_2} 0 0"/>
-      <geometry>
-        <cylinder radius="${wheel_radius}" length="${wheel_width}"/>
-      </geometry>
-    </collision>
-    <xacro:cylinder_inertia m="${wheel_mass}" r="${wheel_radius}" h="${wheel_width}">
-      <origin xyz="0 0 0" rpy="${pi_2} 0.0 0.0"/>
-    </xacro:cylinder_inertia>
-  </link>
-  <!-- ********************** AMR RIGHT WHEEL JOINT *********************************  -->
-  <joint name="amr_RW_joint" type="continuous">
-      <parent link="amr_base"/>
-      <child link="amr_RW"/>
-      <origin xyz="0.0 ${amr_base_width/2 + wheel_width/2} ${-wheel_zoff}" rpy="0 0 0"/>
-      <axis xyz="0 1 0"/>
-  </joint>
-  <!-- ********************** AMR RIGHT WHEEL *********************************  -->
-  <link name="amr_RW">
-    <visual>
-      <origin xyz="0 0 0" rpy="${pi_2} 0 0"/>
-      <geometry>
-        <cylinder radius="${wheel_radius}" length="${wheel_width}"/>
-      </geometry>
-      <material name="red" />
-    </visual>
-    <collision>
-      <origin xyz="0 0 0" rpy="${pi_2} 0 0"/>
-      <geometry>
-        <cylinder radius="${wheel_radius}" length="${wheel_width}"/>
-      </geometry>
-    </collision>
-    <xacro:cylinder_inertia m="${wheel_mass}" r="${wheel_radius}" h="${wheel_width}">
-      <origin xyz="0 0 0" rpy="${pi_2} 0.0 0.0"/>
-    </xacro:cylinder_inertia>
-  </link>
-  <!-- *********************** FRONT CASTER WHEEL JOINT ******************************  -->
-  <joint name="back_caster_joint" type="fixed">
-    <parent link="amr_base"/>
-    <child link="front_caster"/>
-    <origin xyz="${amr_base_length/3} 0.0 ${-(amr_base_height/2)}" rpy="0 0 0"/>
-  </joint>
-  <!-- *********************** FRONT CASTER WHEEL ******************************  -->
-  <link name="front_caster">
-    <visual>
-      <geometry>
-        <sphere radius="${(wheel_radius+wheel_zoff-(amr_base_height/2))}"/>
-      </geometry>
-      <material name="white" />
-    </visual>
-    <collision>
+    <inertial>
+      <mass value="0.114" />
       <origin xyz="0 0 0" rpy="0 0 0"/>
-      <geometry>
-        <sphere radius="${(wheel_radius+wheel_zoff-(amr_base_height/2))}"/>
-      </geometry>
-    </collision>
-    <xacro:sphere_inertia m="${caster_wheel_mass}" r="${(wheel_radius+wheel_zoff-(amr_base_height/2))}">
-      <origin xyz="0 0 0" rpy="${pi_2} 0 ${pi_2}"/>
-    </xacro:sphere_inertia>
-  </link>
-  <!-- *********************** REAR CASTER WHEEL JOINT ******************************  -->
-  <joint name="rear_caster_joint" type="fixed">
-    <parent link="amr_base"/>
-    <child link="rear_caster"/>
-    <origin xyz="${-amr_base_length/3} 0.0 ${-(amr_base_height/2)}" rpy="0 0 0"/>
-  </joint>
-  <!-- *********************** REAR CASTER WHEEL ******************************  -->
-  <link name="rear_caster">
-    <visual>
-      <geometry>
-        <sphere radius="${(wheel_radius+wheel_zoff-(amr_base_height/2))}"/>
-      </geometry>
-      <material name="white" />
-    </visual>
-    <collision>
-      <origin xyz="0 0 0" rpy="0 0 0"/>
-      <geometry>
-        <sphere radius="${(wheel_radius+wheel_zoff-(amr_base_height/2))}"/>
-      </geometry>
-    </collision>
-    <xacro:sphere_inertia m="${caster_wheel_mass}" r="${(wheel_radius+wheel_zoff-(amr_base_height/2))}">
-      <origin xyz="0 0 0" rpy="${pi_2} 0 ${pi_2}"/>
-    </xacro:sphere_inertia>
-  </link>
-  <!-- ****************************** LIDAR JOINT *****************************    -->
-  <joint name="lidar_joint" type="fixed">
-    <parent link="amr_base"/>
-    <child link="lidar"/>
-    <origin xyz="0 0 ${wheel_radius-wheel_zoff+(lidar_height/2)}" rpy="0 0 0"/>
-  </joint>
-  <!-- ****************************** LIDAR *****************************    -->
-  <link name="lidar">
-    <visual>
-      <origin xyz="0 0 0" rpy="0 0 0"/>
-      <geometry>
-        <cylinder radius="${lidar_radius}" length="${lidar_height}"/>
-      </geometry>
-      <material name="red" />
-    </visual>
-    <collision>
-      <origin xyz="0 0 0" rpy="0 0 0"/>
-      <geometry>
-        <cylinder radius="${lidar_radius}" length="${lidar_height}"/>
-      </geometry>
-    </collision>
-    <xacro:cylinder_inertia m="${lidar_mass}" r="${lidar_radius}" h="${lidar_height}">
-      <origin xyz="0 0 0" rpy="0 0 0"/>
-    </xacro:cylinder_inertia>
+      <inertia ixx="0.001" ixy="0" ixz="0" iyy="0.001" iyz="0" izz="0.001" />
+    </inertial>
   </link>
 </robot>

Commit message: fix: diff-drive renewal description

File: amr_description/models/amr/amr.xacro (robot description, xacro)
@@ -3,8 +3,8 @@
 *****************************************************************************************
 *
-*  Filename:			  amr.xacro
-*  Created:				  08/01/2024
-*  Last Modified:	  15/03/2024
-*  Author:				  Archit Jain
+*  Filename:			    amr.xacro
+*  Created:				    08/01/2024
+*  Last Modified:	    15/03/2024
+*  Author:				    Archit Jain
 *
 *****************************************************************************************
@@ -15,12 +15,12 @@
   <xacro:include filename="$(find amr_description)/models/amr/materials.xacro" />
   <!-- ****************** ROBOT CONSTANTS *******************************  -->
-  <xacro:property name="base_width" value="0.39"/>
-  <xacro:property name="base_length" value="0.70"/>
-  <xacro:property name="base_height" value="0.20"/>
-  <xacro:property name="wheel_radius" value="0.14"/>
-  <xacro:property name="wheel_width" value="0.06"/>
-  <xacro:property name="wheel_ygap" value="0.035"/>
-  <xacro:property name="wheel_zoff" value="0.05"/>
-  <xacro:property name="wheel_xoff" value="0.221"/>
+  <xacro:property name="base_width" value="0.40"/>
+  <xacro:property name="base_length" value="0.40"/>
+  <xacro:property name="base_height" value="0.05"/>
+  <xacro:property name="wheel_radius" value="0.04"/>
+  <xacro:property name="wheel_width" value="0.015"/>
+  <xacro:property name="wheel_ygap" value="0.01"/>
+  <xacro:property name="wheel_zoff" value="0.0"/>
+  <xacro:property name="wheel_xoff" value="0.15"/>
   <!-- ****************** INERTIAL PROPERTY MACROS *******************************  -->
   <xacro:macro name="box_inertia" params="m w h d">
@@ -54,5 +54,5 @@
   <link name="base_link">
     <visual>
-      <origin xyz="0 0 -0.05" rpy="1.5707963267949 0 3.141592654"/>
+      <origin xyz="0 0 0" rpy="1.5707963267949 0 3.141592654"/>
       <geometry>
         <box size="${base_length} ${base_height} ${base_width}"/>
@@ -60,9 +60,10 @@
     </visual>
     <collision>
+      <!-- <origin xyz="0 0 0" rpy="1.5707963267949 0 3.141592654"/> -->
       <geometry>
         <box size="${base_length} ${base_width} ${base_height}"/>
       </geometry>
     </collision>
-    <xacro:box_inertia m="40.0" w="${base_width}" d="${base_length}" h="${base_height}"/>
+    <xacro:box_inertia m="1500.0" w="${base_width}" d="${base_length}" h="${base_height}"/>
   </link>
   <!-- *********************** DRIVE WHEELS ******************************  -->
@@ -81,12 +82,12 @@
         </geometry>
       </collision>
-      <xacro:cylinder_inertia m="110.5" r="${wheel_radius}" h="${wheel_width}"/>
+      <xacro:cylinder_inertia m="150.0" r="${wheel_radius}" h="${wheel_width}"/>
     </link>
-    <joint name="${prefix}_joint" type="revolute">
+    <joint name="${prefix}_joint" type="continuous">
       <parent link="base_link"/>
       <child link="${prefix}_link"/>
       <origin xyz="${x_reflect*wheel_xoff} ${y_reflect*(base_width/2+wheel_ygap)} ${-wheel_zoff}" rpy="0 0 0"/>
-      <limit upper="3.1415" lower="-3.1415" effort="30" velocity="5.0"/>
-      <axis xyz="0 1 0"/>
+      <!-- <limit upper="3.1415" lower="-3.1415" effort="30" velocity="5.0"/> -->
+      <axis xyz="0 ${y_reflect} 0"/>
     </joint>
   </xacro:macro>
@@ -99,5 +100,5 @@
     <parent link="base_link"/>
     <child link="imu_link"/>
-    <origin xyz="-0.10 0 0.05" rpy="0 0 0"/>
+    <origin xyz="0.0 0 0.05" rpy="0 0 0"/>
   </joint>
   <link name="imu_link"/>
@@ -106,5 +107,5 @@
     <parent link="base_link"/>
     <child link="lidar_link"/>
-    <origin xyz="0.215 0 0.11" rpy="0 0 0"/>
+    <origin xyz="0.15 0 0.05" rpy="0 0 0"/>
   </joint>
   <link name="lidar_link">
@@ -112,5 +113,5 @@
      <origin xyz="0 0 0" rpy="0 0 0"/>
      <geometry>
-      <cylinder radius="0.0508" length="0.12"/>
+      <cylinder radius="0.025" length="0.05"/>
      </geometry>
     </collision>
@@ -118,9 +119,9 @@
      <origin xyz="0 0 0" rpy="0 0 0"/>
      <geometry>
-      <cylinder radius="0.0508" length="0.12"/>
+      <cylinder radius="0.025" length="0.05"/>
      </geometry>
     </visual>
     <inertial>
-      <mass value="0.114" />
+      <mass value="0.100" />
       <origin xyz="0 0 0" rpy="0 0 0"/>
       <inertia ixx="0.001" ixy="0" ixz="0" iyy="0.001" iyz="0" izz="0.001" />
